Commit message: LaikaGo Working (no Foot Contact)

File: rs_description/urdf/laikago_xacros/leg.xacro (robot description, xacro)
@@ -1,5 +1,5 @@
 <?xml version="1.0"?>
 <robot xmlns:xacro="http://www.ros.org/wiki/xacro">
-    <xacro:include filename="$(find laikago_description)/xacro/transmission.xacro"/>
+    <xacro:include filename="$(find rs_description)/urdf/laikago_xacros/transmission.xacro"/>
     <xacro:macro name="leg" params="name mirror mirror_dae front_hind front_hind_dae *origin">
         <joint name="${name}_hip_joint" type="revolute">
@@ -31,5 +31,5 @@
                 </xacro:if>
                 <geometry>
-                    <mesh filename="package://laikago_description/meshes/hip.dae" scale="1 1 1"/>
+                    <mesh filename="package://rs_description/meshes/laikago_meshes/hip.dae" scale="1 1 1"/>
                 </geometry>
                 <material name="orange"/>
@@ -77,8 +77,8 @@
                 <geometry>
                     <xacro:if value="${mirror_dae == True}">
-                        <mesh filename="package://laikago_description/meshes/thigh.dae" scale="1 1 1"/>
+                        <mesh filename="package://rs_description/meshes/laikago_meshes/thigh.dae" scale="1 1 1"/>
                     </xacro:if>
                     <xacro:if value="${mirror_dae == False}">
-                        <mesh filename="package://laikago_description/meshes/thigh_mirror.dae" scale="1 1 1"/>
+                        <mesh filename="package://rs_description/meshes/laikago_meshes/thigh_mirror.dae" scale="1 1 1"/>
                     </xacro:if>
                 </geometry>
@@ -112,5 +112,5 @@
                 <origin rpy="0 0 0" xyz="0 0 0"/>
                 <geometry>
-                    <mesh filename="package://laikago_description/meshes/calf.dae" scale="1 1 1"/>
+                    <mesh filename="package://rs_description/meshes/laikago_meshes/calf.dae" scale="1 1 1"/>
                 </geometry>
                 <material name="orange"/>

File: rs_description/urdf/laikago_xacros/robot.xacro (robot description, xacro)
@@ -1,8 +1,8 @@
 <?xml version="1.0"?>
 <robot name="laikago_description" xmlns:xacro="http://www.ros.org/wiki/xacro">
-    <xacro:include filename="$(find laikago_description)/xacro/const.xacro"/>
-    <xacro:include filename="$(find laikago_description)/xacro/materials.xacro"/>
-    <xacro:include filename="$(find laikago_description)/xacro/leg.xacro"/>
-    <xacro:include filename="$(find laikago_gazebo)/launch/gazebo.xacro"/>
+    <xacro:include filename="$(find rs_description)/urdf/laikago_xacros/const.xacro"/>
+    <xacro:include filename="$(find rs_description)/urdf/laikago_xacros/materials.xacro"/>
+    <xacro:include filename="$(find rs_description)/urdf/laikago_xacros/leg.xacro"/>
+    <xacro:include filename="$(find rs_description)/urdf/laikago_xacros/gazebo.xacro"/>
     <!-- Rollover Protection mode will add an additional stick on the top, use "true" or "false" to switch it. -->
     <xacro:property name="rolloverProtection" value="false"/>
@@ -33,5 +33,5 @@
             <origin rpy="0 0 0" xyz="0 0 0"/>
             <geometry>
-                <mesh filename="package://laikago_description/meshes/trunk.dae" scale="1 1 1"/>
+                <mesh filename="package://rs_description/meshes/laikago_meshes/trunk.dae" scale="1 1 1"/>
             </geometry>
             <material name="orange"/>
